File: hw/board/hdmi.kicad_pcb (KiCad board)
At the start: 4 copper layers, 77 x 30 mm, 37 parts, among them J1 USB_C_Receptacle_USB2.0_16P, J2 HDMI_A, J3 HDMI_A, SW1 BOOT, SW2 RESET, SW3 FW RESET, U1 USBLC6-2SC6, U2 ESP32-S3-WROOM-2, U3 LM1117DT-3.3

Commit message: XIAO ESP32-S3 based board
Parts:
- removed the C1 at (103.6, 103.3)
- removed C2, C3: 100nF, Capacitor_SMD:C_01005_0402Metric
- removed C4: 1uF, Capacitor_SMD:C_0603_1608Metric
- removed C5, C6: 22uF, Capacitor_SMD:C_0805_2012Metric
- removed the D1 at (125.7, 95.0)
- removed the D2 at (120.0, 79.6)
- removed the D3 at (125.2, 91.8)
- removed D6: GREEN, LED_SMD:LED_0603_1608Metric
- removed F1: Polyfuse 1A, Fuse:Fuse_1206_3216Metric
- removed FB1: BLM21PG220, Inductor_SMD:L_0805_2012Metric
- removed the J1 at (132.1, 102.3)
- removed the R1 at (126.6, 92.0)
- removed the R2 at (121.4, 97.2)
- removed the R3 at (140.6, 96.0)
- removed R4: 5.1K, Resistor_SMD:R_0603_1608Metric
- removed R7: 1K, Resistor_SMD:R_0603_1608Metric
- removed the SW1 at (124.3, 80.0)
- removed SW2: RESET, Button_Switch_SMD:SW_SPST_B3U-1000P
- removed U2: ESP32-S3-WROOM-2, RF_Module:ESP32-S3-WROOM-2
- removed U3: LM1117DT-3.3, Package_TO_SOT_SMD:SOT-223-3_TabPin2
- U1: value USBLC6-2SC6 -> XIAO-ESP32-S3-SMD; footprint Package_TO_SOT_SMD:SOT-23-6 -> Seeed_Studio_XIAO_Series:XIAO-ESP32-S3-SMD
- moved U1 8.34 mm to (138.0, 99.9)
- renumbered C7 to C1, D4 to D1, D5 to D2, D7 to D3, J2 to J1, J3 to J2, R5 to R1, R6 to R2, R8 to R3, SW3 to SW1
Connections:
- U1 pad 1: /D+ -> /HDMI_CEC_0
- U1 pad 2: GND -> /HDMI_CEC_1
- U1 pad 3: /D- -> unconnected-(U1-D2-Pad3)
- U1 pad 4: /USB_D- -> /FIRMWARE_RESET
- U1 pad 5: +5V -> unconnected-(U1-D4-Pad5)
- U1 pad 6: /USB_D+ -> unconnected-(U1-D5-Pad6)
Routing:
- net /FIRMWARE_RESET: track 61.4 -> 28.6 mm
- net Net-(D3-A2): track 32.1 -> 0.00 mm, vias 2 -> 0
- net /HDMI_CEC_1: track 72.8 -> 43.9 mm, vias 3 -> 1
- net /USB_D-: track 24.4 -> 0.00 mm
- net /USB_D+: track 22.0 -> 0.00 mm
- net +5V: track 17.0 -> 0.00 mm
- net +3V3: track 23.0 -> 40.0 mm, vias 8 -> 3
- net /CC1: track 15.4 -> 0.00 mm
- net Net-(F1-Pad1): track 13.8 -> 0.00 mm, vias 2 -> 0
- net /D-: track 11.9 -> 0.00 mm, vias 2 -> 0
- net /D+: track 8.26 -> 0.00 mm, vias 2 -> 0
- net /CC2: track 6.04 -> 0.00 mm
- net Net-(D2-A2): track 5.88 -> 0.00 mm
- net /HDMI_CEC_0: track 62.0 -> 65.4 mm
- net Net-(U2-IO3): track 2.23 -> 0.00 mm
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- removed copper zone on In2.Cu, net +3V3
Other:
- board size 77 x 30 mm -> 60 x 30 mm
