File: hw/board/hdmi.kicad_sch (KiCad schematic)
At the start: 37 parts, among them J1 USB_C_Receptacle_USB2.0_16P, J2 HDMI_A, J3 HDMI_A, SW1 BOOT, SW2 RESET, SW3 FW RESET, U1 USBLC6-2SC6, U2 ESP32-S3-WROOM-2, U3 LM1117DT-3.3

Commit message: XIAO ESP32-S3 based board
Parts:
- removed C1: 10uF, Capacitor_SMD:C_0603_1608Metric, symbol Device:C_Small
- removed C2, C3: 100nF, Capacitor_SMD:C_01005_0402Metric, symbol Device:C_Small
- removed C4: 1uF, Capacitor_SMD:C_0603_1608Metric, symbol Device:C_Small
- removed C5, C6: 22uF, Capacitor_SMD:C_0805_2012Metric, symbol Device:C_Small
- removed D1: 1N5817, Diode_SMD:D_SOD-123, symbol Diode:1N5817
- removed D2, D3: ESD3.3, Diode_SMD:D_SOD-923, symbol Diode:ESD9B3.3ST5G
- removed D6: GREEN, LED_SMD:LED_0603_1608Metric, symbol Device:LED_Small
- removed F1: Polyfuse 1A, Fuse:Fuse_1206_3216Metric, symbol Device:Polyfuse
- removed FB1: BLM21PG220, Inductor_SMD:L_0805_2012Metric, symbol Device:FerriteBead_Small
- removed J1: USB_C_Receptacle_USB2.0_16P, Connector_USB:USB_C_Receptacle_GCT_USB4105-xx-A_16P_TopMnt_Horizontal, symbol Connector:USB_C_Receptacle_USB2.0_16P
- removed R1, R2: 10K, Resistor_SMD:R_0603_1608Metric, symbol Device:R_Small_US
- removed R3, R4: 5.1K, Resistor_SMD:R_0603_1608Metric, symbol Device:R_Small_US
- removed R7: 1K, Resistor_SMD:R_0603_1608Metric, symbol Device:R_Small_US
- removed SW1: BOOT, Button_Switch_SMD:SW_SPST_B3U-1000P, symbol Switch:SW_SPST
- removed SW2: RESET, Button_Switch_SMD:SW_SPST_B3U-1000P, symbol Switch:SW_SPST
- removed U1: USBLC6-2SC6, Package_TO_SOT_SMD:SOT-23-6, symbol Power_Protection:USBLC6-2SC6
- removed U3: LM1117DT-3.3, Package_TO_SOT_SMD:SOT-223-3_TabPin2, symbol Regulator_Linear:LM1117DT-3.3
- C1: renamed from C7; Dielectric (none) -> X7R; MPN (none) -> C1608X7R1C105K080AC; Manufacturer (none) -> TDK; Tolerance (none) -> 10%; Voltage Rating (none) -> 16 V
- D1: renamed from D4; MPN (none) -> TS4148 RCG; Manufacturer (none) -> Taiwan Semiconductor
- D2: renamed from D5; MPN (none) -> TS4148 RCG; Manufacturer (none) -> Taiwan Semiconductor
- D3: renamed from D7; MPN (none) -> ESD9B3.3ST5G; Manufacturer (none) -> onsemi
- J1: renamed from J2; MPN (none) -> 10029449-001RLF; Manufacturer (none) -> Amphenol Communications Solutions
- J2: renamed from J3; MPN (none) -> 10029449-001RLF; Manufacturer (none) -> Amphenol Communications Solutions
- R1: renamed from R5; MPN (none) -> CR0603-JW-273ELF; Manufacturer (none) -> Bourns; Power Rating (none) -> 0.1 W; Tolerance (none) -> 5%
- R2: renamed from R6; MPN (none) -> CR0603-JW-273ELF; Manufacturer (none) -> Bourns; Power Rating (none) -> 0.1 W; Tolerance (none) -> 5%
- R3: renamed from R8; MPN (none) -> CR0603-FX-1002ELF; Manufacturer (none) -> Bourns; Power Rating (none) -> 0.1 W; Tolerance (none) -> 1%
- SW1: renamed from SW3; MPN (none) -> B3U-1000P; Manufacturer (none) -> Omron Electronic Components
- U1: renamed from U2; value ESP32-S3-WROOM-2 -> XIAO-ESP32-S3-SMD; footprint RF_Module:ESP32-S3-WROOM-2 -> Seeed_Studio_XIAO_Series:XIAO-ESP32-S3-SMD; symbol RF_Module:ESP32-S3-WROOM-2 -> Seeed_Studio_XIAO_Series:XIAO-ESP32-S3-SMD; MPN (none) -> 113991114; Manufacturer (none) -> Seeed Studio
Connections:
- net USB_D- is gone; now on net GND: U1.13 (GND)
- net +3V3: now also U1.12 (3V3_OUT); no longer U1.2 (3V3)
- net FIRMWARE_RESET: now also U1.4 (D3); no longer U1.5 (IO5)
- net GND: now also U1.18 (GND), U1.24 (GND), U1.25 (PAD); no longer U1.1 (GND), U1.40 (GND), U1.41 (GND)
- net HDMI_CEC_0: now also U1.1 (D0); no longer U1.39 (IO1)
- net HDMI_CEC_1: now also U1.2 (D1); no longer U1.38 (IO2)
- net USB_D+: no longer names the net of U1.14 (VBUS)
- no-connect marks 28 -> 17
Other:
- note added: "D0 / GPIO1: HDMI_CEC_0 D1 / GPIO2: HDMI_CEC_1"
- note added: "D3 / GPIO4: FIRMWARE_RESET; SW1 retains the firmware reset function."
- note added: "SEEED STUDIO XIAO ESP32-S3"
- note added: "USB-C power, programming, BOOT and RESET are on the XIAO."
- note removed: "ESP32-S3 MODULE"
- note removed: "LDO"
- note removed: "USB-C"
